Commit message: feat(spec): IMU and GNSS frames are imu_link and gnss_link
The Model 3's IMU and GNSS frames carried CARLA's names (carla/imu_link,
carla/gnss_link), kept from csb_isaac until integration. They are now
simulator-neutral, as in Autoware's sample kit (gnss_link): frames imu_link and
gnss_link, topics /sensing/imu/imu_link/imu_raw and
/sensing/gnss/gnss_link/nav_sat_fix. acb renames its own in step, so the two
bridges keep publishing the same frames and topics.

Nothing in Autoware 1.5.0 assumes a vendor/imu_link form: imu_corrector and
gyro_odometer transform through TF from the message's frame_id, and gnss_poser
looks up base_link -> the NavSatFix's frame.

The sensor kit's imu.launch.xml and gnss.launch.xml take the topics as
arguments (imu_raw_name, gnss_fix_name, as Autoware's sample kit does) instead
of hardcoding them twice; test_rig checks the defaults are the rig's.

Regenerated with `just generate`.

Co-Authored-By: Claude Opus 5.5 <noreply@anthropic.com>
Claude-Session: https://claude.ai/code/session_01XsykZth51hsT5oMxxVHcNK

File: src/aib_sensor_kit_launch/aib_sensor_kit_description/urdf/sensor_kit.xacro (robot description, xacro)
@@ -41,20 +41,20 @@
     </joint>
     <link name="camera6/camera_optical_link"/>
-    <!-- imu: imu, published in carla/imu_link on /sensing/imu/carla/imu_link/imu_raw -->
-    <joint name="carla_imu_link_joint" type="fixed">
-      <origin xyz="${calibration['sensor_kit_base_link']['carla/imu_link']['x']} ${calibration['sensor_kit_base_link']['carla/imu_link']['y']} ${calibration['sensor_kit_base_link']['carla/imu_link']['z']}"
-              rpy="${calibration['sensor_kit_base_link']['carla/imu_link']['roll']} ${calibration['sensor_kit_base_link']['carla/imu_link']['pitch']} ${calibration['sensor_kit_base_link']['carla/imu_link']['yaw']}"/>
+    <!-- imu: imu, published in imu_link on /sensing/imu/imu_link/imu_raw -->
+    <joint name="imu_link_joint" type="fixed">
+      <origin xyz="${calibration['sensor_kit_base_link']['imu_link']['x']} ${calibration['sensor_kit_base_link']['imu_link']['y']} ${calibration['sensor_kit_base_link']['imu_link']['z']}"
+              rpy="${calibration['sensor_kit_base_link']['imu_link']['roll']} ${calibration['sensor_kit_base_link']['imu_link']['pitch']} ${calibration['sensor_kit_base_link']['imu_link']['yaw']}"/>
       <parent link="sensor_kit_base_link"/>
-      <child link="carla/imu_link"/>
+      <child link="imu_link"/>
     </joint>
-    <link name="carla/imu_link"/>
-    <!-- gnss: gnss, published in carla/gnss_link on /sensing/gnss/carla/gnss_link/nav_sat_fix -->
-    <joint name="carla_gnss_link_joint" type="fixed">
-      <origin xyz="${calibration['sensor_kit_base_link']['carla/gnss_link']['x']} ${calibration['sensor_kit_base_link']['carla/gnss_link']['y']} ${calibration['sensor_kit_base_link']['carla/gnss_link']['z']}"
-              rpy="${calibration['sensor_kit_base_link']['carla/gnss_link']['roll']} ${calibration['sensor_kit_base_link']['carla/gnss_link']['pitch']} ${calibration['sensor_kit_base_link']['carla/gnss_link']['yaw']}"/>
+    <link name="imu_link"/>
+    <!-- gnss: gnss, published in gnss_link on /sensing/gnss/gnss_link/nav_sat_fix -->
+    <joint name="gnss_link_joint" type="fixed">
+      <origin xyz="${calibration['sensor_kit_base_link']['gnss_link']['x']} ${calibration['sensor_kit_base_link']['gnss_link']['y']} ${calibration['sensor_kit_base_link']['gnss_link']['z']}"
+              rpy="${calibration['sensor_kit_base_link']['gnss_link']['roll']} ${calibration['sensor_kit_base_link']['gnss_link']['pitch']} ${calibration['sensor_kit_base_link']['gnss_link']['yaw']}"/>
       <parent link="sensor_kit_base_link"/>
-      <child link="carla/gnss_link"/>
+      <child link="gnss_link"/>
     </joint>
-    <link name="carla/gnss_link"/>
+    <link name="gnss_link"/>
   </xacro:macro>
 </robot>
